Commit message: firist step for update

File: mir_description/urdf/include/common.gazebo.xacro (robot description, xacro)
@@ -3,11 +3,11 @@
   <xacro:macro name="controller_plugin_gazebo" params="robot_namespace">
     <gazebo>
-      <plugin filename="libgazebo_ros2_control.so" name="gazebo_ros2_control">
-        <robot_param>robot_description</robot_param>
-        <robot_param_node>robot_state_publisher</robot_param_node>
+      <!-- Usando o plugin nativo do Gazebo Harmonic para controle -->
+      <plugin filename="gz-sim-joint-controller-system" name="gz::sim::systems::JointController">
+        <robot_description>robot_description</robot_description>
         <xacro:unless value="${robot_namespace == ''}">
           <robot_namespace>${robot_namespace}</robot_namespace>
         </xacro:unless>
-        <control_period>0.001</control_period>
+        <update_rate>1000</update_rate>
       </plugin>
     </gazebo>

File: mir_description/urdf/include/imu.gazebo.urdf.xacro (robot description, xacro)
@@ -71,12 +71,8 @@
           </linear_acceleration>
         </imu>
-        <plugin filename="libgazebo_ros_imu_sensor.so" name="imu_plugin">
-        <initial_orientation_as_reference>false</initial_orientation_as_reference>
-          <ros>
-            <namespace>${imu_topic}</namespace>
-            <remapping>~/out:=data</remapping>
-            <frame_name>${imu_frame}</frame_name>  <!-- from real MiR -->
-          </ros>
-        </plugin>
+        <!-- Usando sensor IMU nativo do Gazebo Harmonic -->
+        <topic>${imu_topic}/data</topic>
+        <!-- Removendo parâmetros não suportados pelo SDF -->
+        <!-- frame_name não é suportado diretamente no elemento sensor no SDF -->
       </sensor>
     </gazebo>

File: mir_description/urdf/include/mir.gazebo.xacro (robot description, xacro)
@@ -1,35 +1,29 @@
 <?xml version="1.0"?>
 <robot xmlns:xacro="http://ros.org/wiki/xacro">
-  <!-- See https://github.com/ros-simulation/gazebo_ros_pkgs/wiki/ROS-2-Migration:-Diff-drive for ros2 information -->
+  <!-- See https://github.com/gazebo-release/gz_ros2_control for ros2 information -->
   <xacro:macro name="diff_controller_plugin_gazebo" params="prefix ns left_wheel_joint right_wheel_joint wheel_separation wheel_radius">
     <gazebo>
-      <!-- Use gazebo_ros_joint_state_publisher instead of publishWheelJointState -->
-      <plugin name="joint_states" filename="libgazebo_ros_joint_state_publisher.so">
-        <ros>
-          <namespace>${ns}</namespace>
-        </ros>
-        <update_rate>1000.0</update_rate>
+      <!-- Atualizado para usar o plugin nativo do Gazebo Harmonic -->
+      <plugin filename="gz-sim-joint-state-publisher-system" name="gz::sim::systems::JointStatePublisher">
+        <topic>joint_states</topic>
         <joint_name>${right_wheel_joint}</joint_name>
         <joint_name>${left_wheel_joint}</joint_name>
       </plugin>
-      <plugin name="diff_drive_controller" filename="libgazebo_ros_diff_drive.so">
-        <ros>
-          <remapping>cmd_vel:=${prefix}cmd_vel</remapping>
-          <remapping>odom:=${prefix}odom</remapping>
-        </ros>
-        <legacy_mode>false</legacy_mode>
-        <always_on>true</always_on>
-        <update_rate>1000.0</update_rate>
+      <!-- Substituído pelo plugin nativo do Gazebo Harmonic conforme documentação oficial -->
+      <plugin filename="gz-sim-diff-drive-system" name="gz::sim::systems::DiffDrive">
+        <!-- wheels -->
         <left_joint>${left_wheel_joint}</left_joint>
         <right_joint>${right_wheel_joint}</right_joint>
+        <!-- kinematics -->
         <wheel_separation>${wheel_separation}</wheel_separation>
-        <wheel_diameter>${2*wheel_radius}</wheel_diameter>
-        <odometry_frame>${prefix}odom</odometry_frame>
-        <robot_base_frame>${prefix}base_footprint</robot_base_frame>
-        <publish_odom>true</publish_odom>
-        <publish_wheel_tf>false</publish_wheel_tf>
-        <publish_odom_tf>true</publish_odom_tf>
-        <max_wheel_torque>10</max_wheel_torque>
-        <max_wheel_acceleration>2.8</max_wheel_acceleration>
+        <wheel_radius>${wheel_radius}</wheel_radius>
+        <!-- limits -->
+        <max_linear_acceleration>2.8</max_linear_acceleration>
+        <topic>${prefix}cmd_vel</topic>
+        <odom_topic>${prefix}odom</odom_topic>
+        <frame_id>${prefix}odom</frame_id>
+        <child_frame_id>${prefix}base_footprint</child_frame_id>
+        <odom_publisher_frequency>30</odom_publisher_frequency>
+        <tf_topic>tf</tf_topic>
       </plugin>
     </gazebo>
@@ -52,18 +46,14 @@
     <xacro:set_wheel_friction link="${prefix}br_caster_wheel_link" friction="1"/>
   </xacro:macro>
- <!-- See https://github.com/ros-simulation/gazebo_ros_pkgs/wiki/ROS-2-Migration:-P3D for ros2 information -->
   <xacro:macro name="p3d_base_controller" params="prefix">
     <gazebo>
-      <plugin name="p3d_base_controller" filename="libgazebo_ros_p3d.so">
-        <ros>
-          <remapping>odom:=${prefix}base_pose_ground_truth</remapping>
-        </ros>
-        <always_on>true</always_on>
+      <!-- Usando o plugin nativo do Gazebo Harmonic para odometria -->
+      <plugin filename="gz-sim-odometry-publisher-system" name="gz::sim::systems::OdometryPublisher">
+        <odom_topic>${prefix}base_pose_ground_truth</odom_topic>
+        <odom_frame>map</odom_frame>
+        <robot_base_frame>${prefix}base_footprint</robot_base_frame>
+        <dimensions>3</dimensions>
+        <gaussian_noise>0.01</gaussian_noise>
         <update_rate>50.0</update_rate>
-        <body_name>${prefix}base_footprint</body_name>
-        <gaussian_noise>0.01</gaussian_noise>
-        <frame_name>map</frame_name>
-        <xyz_offset>0 0 0</xyz_offset>
-        <rpy_offset>0 0 0</rpy_offset>
       </plugin>
     </gazebo>

File: mir_description/urdf/include/mir_v1.urdf.xacro (robot description, xacro)
@@ -8,4 +8,5 @@
   <xacro:include filename="$(find mir_description)/urdf/include/mir.transmission.xacro" />
   <xacro:include filename="$(find mir_description)/urdf/include/sick_s300.urdf.xacro" />
+  <xacro:include filename="$(find mir_description)/urdf/include/gz_ros2_control.xacro" />
   <xacro:property name="deg_to_rad" value="0.017453293" />
   <xacro:property name="mir_base_mass" value="58.0" />
@@ -70,9 +71,6 @@
     </joint>
     <gazebo>
-      <plugin name="${locationprefix}_caster_rotation_joint_states" filename="libgazebo_ros_joint_state_publisher.so">
-        <ros>
-          <namespace>${ns}</namespace>
-        </ros>
-        <update_rate>200.0</update_rate>
+      <plugin filename="gz-sim-joint-state-publisher-system" name="gz::sim::systems::JointStatePublisher">
+        <topic>${locationprefix}_caster_rotation_joint_states</topic>
         <joint_name>${prefix}${locationprefix}_caster_rotation_joint</joint_name>
       </plugin>
@@ -94,5 +92,6 @@
         <origin xyz="0 0 0" rpy="0 0 0" />
         <geometry>
-          <mesh filename="package://mir_description/meshes/visual/caster_wheel_base.stl" />
+          <!-- Substituindo mesh por geometria simples para compatibilidade com dartsim -->
+          <cylinder radius="0.05" length="0.1"/>
         </geometry>
         <xacro:insert_block name="material_silver" />
@@ -101,5 +100,6 @@
         <origin xyz="0 0 0" rpy="0 0 0" />
         <geometry>
-          <mesh filename="package://mir_description/meshes/collision/caster_wheel_base.stl" />
+          <!-- Substituindo mesh por geometria simples para compatibilidade com dartsim -->
+          <cylinder radius="0.05" length="0.1"/>
         </geometry>
       </collision>
@@ -116,9 +116,6 @@
     </joint>
     <gazebo>
-      <plugin name="${locationprefix}_caster_wheel_joint_states" filename="libgazebo_ros_joint_state_publisher.so">
-        <ros>
-          <namespace>${ns}</namespace>
-        </ros>
-        <update_rate>200.0</update_rate>
+      <plugin filename="gz-sim-joint-state-publisher-system" name="gz::sim::systems::JointStatePublisher">
+        <topic>${locationprefix}_caster_wheel_joint_states</topic>
         <joint_name>${prefix}${locationprefix}_caster_wheel_joint</joint_name>
       </plugin>
@@ -160,5 +157,6 @@
         <origin xyz="${mir_act_wheel_dx} 0 0" rpy="0 0 0" />
         <geometry>
-          <mesh filename="package://mir_description/meshes/visual/${mir_type}_base.stl" />
+          <!-- Substituindo mesh por geometria simples para compatibilidade com dartsim -->
+          <box size="0.9 0.58 0.3"/>
         </geometry>
         <xacro:insert_block name="material_white" />
@@ -167,5 +165,6 @@
         <origin xyz="${mir_act_wheel_dx} 0 0" rpy="0 0 0" />
         <geometry>
-          <mesh filename="package://mir_description/meshes/collision/${mir_type}_base.stl" />
+          <!-- Substituindo mesh por geometria simples para compatibilidade com dartsim -->
+          <box size="0.9 0.58 0.3"/>
         </geometry>
       </collision>
@@ -243,4 +242,6 @@
     <xacro:set_all_wheel_frictions prefix="${prefix}"/>
     <xacro:p3d_base_controller prefix="${prefix}" />
+    <!-- Adiciona o plugin gz_ros2_control para integração com ROS 2 Control -->
+    <xacro:gz_ros2_control prefix="${prefix}" />
   </xacro:macro>
 </robot>

File: mir_description/urdf/include/sick_s300.urdf.xacro (robot description, xacro)
@@ -11,13 +11,16 @@
         <origin xyz="0.0 0.0 0.0" rpy="${pi} 0 0" />
         <geometry>
-          <mesh filename="package://mir_description/meshes/visual/sick_lms-100.stl" />
+          <!-- Substituindo mesh por geometria simples para compatibilidade com dartsim -->
+          <cylinder radius="${laser_y/2}" length="${laser_z}"/>
         </geometry>
-        <!-- <xacro:insert_block name="material_yellow" /> -->
-        <xacro:insert_block name="material_black" />
+        <material name="black">
+          <color rgba="0.0 0.0 0.0 1.0"/>
+        </material>
       </visual>
       <collision>
         <origin xyz="0.0 0.0 0.0" rpy="${pi} 0 0" />
         <geometry>
-          <mesh filename="package://mir_description/meshes/visual/sick_lms-100.stl" />
+          <!-- Substituindo mesh por geometria simples para compatibilidade com dartsim -->
+          <cylinder radius="${laser_y/2}" length="${laser_z}"/>
         </geometry>
       </collision>
@@ -27,7 +30,7 @@
     </link>
     <gazebo reference="${prefix}${link}">
-      <!-- <material value="Gazebo/Yellow" /> -->
-      <material value="Gazebo/FlatBlack" />
-      <sensor type="ray" name="${prefix}${link}">
+      <!-- Usando cores diretas em vez de materiais Ogre -->
+      <material>Gazebo/Black</material>
+      <sensor type="gpu_ray" name="${prefix}${link}">
         <visualize>false</visualize>
         <update_rate>12.5</update_rate>
@@ -55,11 +58,8 @@
           </noise>
         </ray>
-        <plugin name="gazebo_ros_${link}_controller" filename="libgazebo_ros_ray_sensor.so">
-          <ros>
-            <remapping>~/out:=${prefix}${topic}</remapping>
-          </ros>
-          <output_type>sensor_msgs/LaserScan</output_type>
-          <frame_name>${prefix}${link}</frame_name>
-        </plugin>
+        <!-- Usando sensor LIDAR nativo do Gazebo Harmonic -->
+        <topic>${prefix}${topic}</topic>
+        <!-- Removendo parâmetros não suportados pelo SDF -->
+        <!-- frame_name e output_type não são suportados diretamente no elemento sensor no SDF -->
       </sensor>
     </gazebo>

File: urdf/include/mir_v1.urdf.xacro (robot description, xacro)
@@ -70,9 +70,6 @@
     </joint>
     <gazebo>
-      <plugin name="${locationprefix}_caster_rotation_joint_states" filename="libgazebo_ros_joint_state_publisher.so">
-        <ros>
-          <namespace>${ns}</namespace>
-        </ros>
-        <update_rate>200.0</update_rate>
+      <plugin filename="gz-sim-joint-state-publisher-system" name="gz::sim::systems::JointStatePublisher">
+        <topic>${locationprefix}_caster_rotation_joint_states</topic>
         <joint_name>${prefix}${locationprefix}_caster_rotation_joint</joint_name>
       </plugin>
@@ -116,9 +113,6 @@
     </joint>
     <gazebo>
-      <plugin name="${locationprefix}_caster_wheel_joint_states" filename="libgazebo_ros_joint_state_publisher.so">
-        <ros>
-          <namespace>${ns}</namespace>
-        </ros>
-        <update_rate>200.0</update_rate>
+      <plugin filename="gz-sim-joint-state-publisher-system" name="gz::sim::systems::JointStatePublisher">
+        <topic>${locationprefix}_caster_wheel_joint_states</topic>
         <joint_name>${prefix}${locationprefix}_caster_wheel_joint</joint_name>
       </plugin>

File: urdf/include/sick_s300.urdf.xacro (robot description, xacro)
@@ -29,5 +29,5 @@
       <!-- <material value="Gazebo/Yellow" /> -->
       <material value="Gazebo/FlatBlack" />
-      <sensor type="ray" name="${prefix}${link}">
+      <sensor type="gpu_lidar" name="${prefix}${link}">
         <visualize>false</visualize>
         <update_rate>12.5</update_rate>
@@ -55,11 +55,8 @@
           </noise>
         </ray>
-        <plugin name="gazebo_ros_${link}_controller" filename="libgazebo_ros_ray_sensor.so">
-          <ros>
-            <remapping>~/out:=${prefix}${topic}</remapping>
-          </ros>
-          <output_type>sensor_msgs/LaserScan</output_type>
-          <frame_name>${prefix}${link}</frame_name>
-        </plugin>
+        <!-- Usando sensor LIDAR nativo do Gazebo Harmonic -->
+        <topic>${prefix}${topic}</topic>
+        <!-- Removendo parâmetros não suportados pelo SDF -->
+        <!-- frame_name e output_type não são suportados diretamente no elemento sensor no SDF -->
       </sensor>
     </gazebo>
