Commit message: Add ros2_control configuration and map files for Lab4.0

File: mir_description/urdf/include/gz_ros2_control.xacro (robot description, xacro)
@@ -1,5 +1,20 @@
 <?xml version="1.0"?>
-<robot xmlns:xacro="http://ros.org/wiki/xacro">
+<robot xmlns:xacro="http://wiki.ros.org/xacro">  <!-- URI CORRIGIDO AQUI -->
   <xacro:macro name="gz_ros2_control" params="prefix">
+    <ros2_control name="mir" type="system">
+      <hardware>
+        <plugin>gz_ros2_control/GazeboSystem</plugin>
+      </hardware>
+      <joint name="${prefix}left_wheel_joint">
+        <command_interface name="velocity"/>
+        <state_interface name="position"/>
+        <state_interface name="velocity"/>
+      </joint>
+      <joint name="${prefix}right_wheel_joint">
+        <command_interface name="velocity"/>
+        <state_interface name="position"/>
+        <state_interface name="velocity"/>
+      </joint>
+    </ros2_control>
     <gazebo>
       <plugin filename="gz-sim-joint-controller-system" name="gz::sim::systems::JointController">
